File: hardware/garage-opener-pcb/garage-opener-pcb.kicad_sch (KiCad schematic)
At the start: 32 parts, among them J1 5V IN, J2 OPENER COM/NO/NC, J3 REED, K1 SRD-05VDC-SL-C, Q1 MMBT2222A, U1 ESP32-DevKitC-V4, U2 DHT22

Commit message: fix(hw): use 1.1 A PTC and require 5.1 V supply for 5 V rail margin
Parts:
- F1: value 0.5A hold -> 1.1A hold
Changed lines of the file:
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@@
 			)
 		)
-		(property "Value" "0.5A hold"
+		(property "Value" "1.1A hold"
 			(at 154.94 48.26 90)
 			(show_name no)

Commit message: feat(hw): redraw schematic with wired circuits; labels only for ESP32 signals
Connections:
- net COIL_LO: no longer names the net of D2.2 (A), K1.2, Q1.3 (C)
- net LED_DOOR_A: no longer names the net of D5.2 (A), R7.2
- net LED_RUN_A: no longer names the net of D4.2 (A), R6.2
- net Q1_BASE: no longer names the net of Q1.1 (B), R1.2
- net REED_EXT: no longer names the net of D3.1 (A1), J3.1 (Pin_1), R4.1
- net RELAY_COM: no longer names the net of J2.1 (Pin_1), K1.1
- net RELAY_NC: no longer names the net of J2.3 (Pin_3), K1.4
- net RELAY_NO: no longer names the net of J2.2 (Pin_2), K1.3
- net VIN_FUSED: no longer names the net of D1.2 (A), F1.2
- net VIN_RAW: no longer names the net of F1.1, J1.1 (Pin_1)
Other:
- note added: "ESP32 DevKitC V4 (WROOM-32U) plugs into 2x 1x19 sockets (U1 footprint)"
- note added: "LEDs: RUN (GPIO2, strapping pin - LED + R to GND is a safe load) and DOOR (GPIO16). ~4 mA each."
- note added: "NOTES 1. Firmware unchanged: GPIO map = main/board.h. Reset/factory button = devkit Boot button (GPIO0). 2. Power J1 from 5.1-5.2 V. External 5 V and USB together only if the devkit has a diode on USB VBUS. 3. Devkit rows are 25.4 mm apart (DevKitC V4) - measure the real board before ordering PCBs. 4. Relay output is for the opener's low-voltage push-button input. Not for mains. 5. Bring-up check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"
- note added: "POWER: 5.1 V in -> PTC fuse -> Schottky (reverse-polarity + USB back-feed block) -> +5V"
- note added: "REED SWITCH (GPIO4): closed = low, open = high. 10k pull-up + 1k/100nF filter (~1 ms) + ESD diode at J3."
- note added: "RELAY (GPIO5): R2 4k7 pull-down holds GPIO5 ~0.3 V during boot (internal ~45k pull-up), below Q1 Vbe -> relay cannot pull in while the ESP32 resets. D2 = flyback diode. J2: wire COM + NO across the opener's wall button (NC spare)."
- note removed: "ESP32 DevKitC V4 (WROOM-32U) - plugs into 2x 1x19 sockets (U1 footprint)"
- note removed: "LEDs: RUN (GPIO2, strapping pin - LED+R to GND is a safe load) and DOOR (GPIO16). ~4 mA each."
- note removed: "NOTES 1. Firmware unchanged: GPIO map = main/board.h. Reset/factory button = devkit Boot button (GPIO0). 2. External 5 V (J1) and USB together only if the devkit has a diode on USB VBUS - check first. 3. Devkit rows are 25.4 mm apart (DevKitC V4) - measure the real board before ordering PCBs. 4. Relay output is for the opener's low-voltage push-button input. Not for mains. 5. Bring-up checklist: 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"
- note removed: "POWER: 5 V in -> PTC fuse -> Schottky (reverse-polarity + USB back-feed block) -> +5V"
- note removed: "REED SWITCH (GPIO4): closed = low, open = high. 10k pull-up + 1k/100nF filter (~1 ms) + ESD at J3."
- note removed: "RELAY (GPIO5): R2 4k7 pull-down holds GPIO5 ~0.3 V during boot (internal ~45k pull-up), below Q1 Vbe -> relay cannot pull in while the ESP32 resets. J2: wire COM+NO across the opener's wall button."
- moved on the sheet: C1, C2, C3, C4, D1, D2, D3, D4, D5, F1, H1, H2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

Commit message: feat(hw): pluggable Phoenix connectors for J1-J3 (3.81 mm power, 5.08 mm relay/reed)
Parts:
- J1: footprint TerminalBlock_Phoenix:TerminalBlock_Phoenix_MKDS-1,5-2_1x02_P5.00mm_Horizontal -> Connector_Phoenix_MC:PhoenixContact_MC_1,5_2-G-3.81_1x02_P3.81mm_Horizontal
- J2: footprint TerminalBlock_Phoenix:TerminalBlock_Phoenix_MKDS-1,5-3_1x03_P5.00mm_Horizontal -> Connector_Phoenix_MSTB:PhoenixContact_MSTBA_2,5_3-G-5,08_1x03_P5.08mm_Horizontal
- J3: footprint TerminalBlock_Phoenix:TerminalBlock_Phoenix_MKDS-1,5-2_1x02_P5.00mm_Horizontal -> Connector_Phoenix_MSTB:PhoenixContact_MSTBA_2,5_2-G-5,08_1x02_P5.08mm_Horizontal
Changed lines of the file:
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@@
 			)
 		)
-		(property "Footprint" "TerminalBlock_Phoenix:TerminalBlock_Phoenix_MKDS-1,5-3_1x03_P5.00mm_Horizontal"
+		(property "Footprint" "Connector_Phoenix_MSTB:PhoenixContact_MSTBA_2,5_3-G-5,08_1x03_P5.08mm_Horizontal"
 			(at 195.58 96.52 0)
 			(hide yes)
@@
 			)
 		)
-		(property "Footprint" "TerminalBlock_Phoenix:TerminalBlock_Phoenix_MKDS-1,5-2_1x02_P5.00mm_Horizontal"
+		(property "Footprint" "Connector_Phoenix_MC:PhoenixContact_MC_1,5_2-G-3.81_1x02_P3.81mm_Horizontal"
 			(at 121.92 50.8 0)
 			(hide yes)
@@
 			)
 		)
-		(property "Footprint" "TerminalBlock_Phoenix:TerminalBlock_Phoenix_MKDS-1,5-2_1x02_P5.00mm_Horizontal"
+		(property "Footprint" "Connector_Phoenix_MSTB:PhoenixContact_MSTBA_2,5_2-G-5,08_1x02_P5.08mm_Horizontal"
 			(at 121.92 157.48 0)
 			(hide yes)
