File: hardware/garage-opener-pcb/garage-opener-pcb.kicad_pcb (KiCad board)
At the start: 2 copper layers, 95 x 70 mm, 32 parts, among them J1 5V IN, J2 OPENER COM/NO/NC, J3 REED, K1 SRD-05VDC-SL-C, Q1 MMBT2222A, U1 ESP32-DevKitC-V4, U2 DHT22

Commit message: feat(hw): route rev 1 PCB with Freerouting; DRC, unconnected and parity clean
Routing:
- net +5V: track 0.00 -> 181.1 mm
- net +3V3: track 0.00 -> 119.0 mm, vias 0 -> 2
- net /RELAY_DRV: track 0.00 -> 57.2 mm, vias 0 -> 1
- net Net-(J2-Pin_1): track 0.00 -> 47.0 mm
- net /DHT_DATA: track 0.00 -> 44.6 mm
- net /REED: track 0.00 -> 31.5 mm
- net Net-(J2-Pin_3): track 0.00 -> 29.4 mm
- net Net-(J2-Pin_2): track 0.00 -> 29.1 mm
- net Net-(D2-A): track 0.00 -> 19.6 mm
- net /LED_DOOR: track 0.00 -> 19.6 mm
- net /BOARD_ID0: track 0.00 -> 18.6 mm
- net Net-(J1-Pin_1): track 0.00 -> 18.3 mm
- net /LED_RUN: track 0.00 -> 16.3 mm
- net Net-(D3-A1): track 0.00 -> 15.2 mm
- net /BOARD_ID1: track 0.00 -> 12.6 mm
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
Commit message: feat(hw): silkscreen labels and Aisler fab outputs (Gerbers, drill, STEP, STL)
Other:
- board text added: "+"
- board text added: "-"
- board text added: "5V IN"
- board text added: "COM"
- board text added: "DOOR"
- board text added: "NC"
- board text added: "NO"
- board text added: "REED"
- board text added: "RUN"
- board text added: "garage-opener"
- board text added: "rev 1"
Changed lines of the file:
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@@
 			(at 1.9 -3 0)
 			(layer "F.SilkS")
+			(hide yes)
 			(effects
 				(font
@@
 		(tags "ESP32 DevKitC socket")
 		(property "Reference" "U1"
-			(at 12.7 -8 270)
+			(at 12.7 21.2 270)
 			(layer "F.SilkS")
 			(effects
@@
 			(at 2.54 -3.2 0)
 			(layer "F.SilkS")
+			(hide yes)
 			(effects
 				(font
@@
 		(tags "resistor")
 		(property "Reference" "R8"
-			(at 0 -1.65 90)
+			(at 3.2 0 0)
 			(layer "F.SilkS")
 			(effects
 				(font
-					(size 1 1)
+					(size 0.8 0.8)
 					(thickness 0.15)
 				)
@@
 			(at 1.27 -2.96 0)
 			(layer "F.SilkS")
+			(hide yes)
 			(effects
 				(font
@@
 		(tags "resistor")
 		(property "Reference" "R9"
-			(at 0 -1.65 90)
+			(at 3.2 0 0)
 			(layer "F.SilkS")
 			(effects
 				(font
-					(size 1 1)
+					(size 0.8 0.8)
 					(thickness 0.15)
 				)
@@
 		(tags "relay Sanyu SRD form C")
 		(property "Reference" "K1"
-			(at 8.1 9.2 270)
+			(at 8.5 0 270)
 			(layer "F.SilkS")
 			(effects
@@
 		(tags "resistor")
 		(property "Reference" "R10"
-			(at 0 -1.65 90)
+			(at 3.2 0 0)
 			(layer "F.SilkS")
 			(effects
 				(font
-					(size 1 1)
+					(size 0.8 0.8)
 					(thickness 0.15)
 				)
@@
 			(at 1.27 -2.96 0)
 			(layer "F.SilkS")
+			(hide yes)
 			(effects
 				(font
@@
 			(at 5.08 -3.2 0)
 			(layer "F.SilkS")
+			(hide yes)
 			(effects
 				(font
@@
 		(tags "resistor")
 		(property "Reference" "R11"
-			(at 0 -1.65 90)
+			(at 3.2 0 0)
 			(layer "F.SilkS")
 			(effects
 				(font
-					(size 1 1)
+					(size 0.8 0.8)
 					(thickness 0.15)
 				)
@@
 		(layer "Edge.Cuts")
 	)
+	(gr_text "RUN"
+		(at 107.27 143 0)
+		(layer "F.SilkS")
+		(effects
+			(font
+				(size 1 1)
+				(thickness 0.15)
+			)
+		)
+	)
+	(gr_text "garage-opener"
+		(at 110 157 0)
+		(layer "F.SilkS")
+		(effects
+			(font
+				(size 1 1)
+				(thickness 0.15)
+			)
+		)
+	)
+	(gr_text "rev 1"
+		(at 110 159 0)
+		(layer "F.SilkS")
+		(effects
+			(font
+				(size 1 1)
+				(thickness 0.15)
+			)
+		)
+	)
+	(gr_text "DOOR"
+		(at 113.77 143 0)
+		(layer "F.SilkS")
+		(effects
+			(font
+				(size 1 1)
+				(thickness 0.15)
+			)
+		)
+	)
+	(gr_text "+"
+		(at 122 158.16 0)
+		(layer "F.SilkS")
+		(effects
+			(font
+				(size 1 1)
+				(thickness 0.15)
+			)
+		)
+	)
+	(gr_text "5V IN"
+		(at 123.905 156.36 0)
+		(layer "F.SilkS")
+		(effects
+			(font
+				(size 1 1)
+				(thickness 0.15)
+			)
+		)
+	)
+	(gr_text "-"
+		(at 125.81 158.16 0)
+		(layer "F.SilkS")
+		(effects
+			(font
+				(size 1 1)
+				(thickness 0.15)
+			)
+		)
+	)
+	(gr_text "REED"
+		(at 142.54 155.56 0)
+		(layer "F.SilkS")
+		(effects
+			(font
+				(size 1 1)
+				(thickness 0.15)
+			)
+		)
+	)
+	(gr_text "COM"
+		(at 158 155.56 0)
+		(layer "F.SilkS")
+		(effects
+			(font
+				(size 1 1)
+				(thickness 0.15)
+			)
+		)
+	)
+	(gr_text "NO"
+		(at 163.08 155.56 0)
+		(layer "F.SilkS")
+		(effects
+			(font
+				(size 1 1)
+				(thickness 0.15)
+			)
+		)
+	)
+	(gr_text "NC"
+		(at 168.16 155.56 0)
+		(layer "F.SilkS")
+		(effects
+			(font
+				(size 1 1)
+				(thickness 0.15)
+			)
+		)
+	)
 	(segment
